File: Hardware/keyboard_matrix.kicad_sch (KiCad schematic)
At the start: 79 parts, among them IC3 TS02-66-80-BK-160-LCR-D, SW1 PEC12R-4125F-S0012

Commit message: updated files, added PDF versions on schematic and PCB
Other:
- note added: "Key matrix"
- note added: "PC audio controls"
- moved on the sheet: C18, C19, C20, C21, IC3, R11, R12, R13, R14, R15, R16, R17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
